File: board/board.sch (KiCad schematic (older format))
At the start: 78 parts, among them IC1 LVC245A, IC2 LVC245A, J1 Conn_01x06_Male, J10 Conn_01x02, J11 Conn_01x05_Male, J2 AudioJack4_Ground, J3 Conn_01x02, J5 Conn_01x01_Male, J6 Conn_01x01_Male, J7 Conn_01x01_Male, J8 Conn_01x01_Male, J9 Conn_01x01_Male, U1 THS7316, U2 10M02SCE144

Commit message: Rework to be manufacturable by JLCPCB
Parts:
- added C26, C28: 100nF, Capacitor_SMD:C_0402_1005Metric, symbol Device:C_Small
- C1, C2, C3, C4, C5: footprint Capacitor_SMD:C_0805_2012Metric_Pad1.15x1.40mm_HandSolder -> Capacitor_SMD:C_0805_2012Metric
- C11, C12, C13, C14, C15, C16, C17, C18, C19, C20, C21, C22, C23, C24, C25, C31, C32, C33, C34, C6, C7, C8, C9: footprint Capacitor_SMD:C_0603_1608Metric_Pad1.05x0.95mm_HandSolder -> Capacitor_SMD:C_0402_1005Metric
- IC1, IC2: symbol Library:LVC245A -> board-rescue:LVC245A-Library
- L1, L2, L3: footprint Capacitor_SMD:C_0805_2012Metric_Pad1.15x1.40mm_HandSolder -> Inductor_SMD:L_0805_2012Metric_Pad1.15x1.40mm_HandSolder
- OSC1: symbol components:LFSPXO024957 -> board-rescue:LFSPXO024957-components
- R1: footprint Resistor_SMD:R_0805_2012Metric_Pad1.15x1.40mm_HandSolder -> Resistor_SMD:R_0603_1608Metric
- R10, R11, R12, R13, R14, R15, R16, R17, R18, R19, R2, R20, R21, R22, R23, R24, R25, R26, R27, R28, R29, R3, R4, R5, R6, R7, R8, R9: footprint Resistor_SMD:R_0805_2012Metric_Pad1.15x1.40mm_HandSolder -> Resistor_SMD:R_0402_1005Metric
- REG1: symbol components:LM1117IMPX-3.3 -> board-rescue:LM1117IMPX-3.3-components
- U1: symbol Library:THS7316 -> board-rescue:THS7316-Library
- U2: symbol components:10M02SCE144 -> board-rescue:10M02SCE144-components
Connections:
- wire segments 431 -> 439
- no-connect marks 68 -> 69
Other:
- moved on the sheet: C31, C32, C33, C34
